File: High Power SW.sch (KiCad schematic (older format))
At the start: 15 parts, among them CN1 Jumper_NC_Small, Q1 IRFR7540TRPBF, U1 PS2801C-1-A

Commit message: Update Board to have new input opto
Gerber files are not built yet
Parts:
- removed BED+1, BED-1, POWER+1: CONN_01X01, MyLib:Keystone_4966, symbol CONN_01X01
- added BED+, BED-, POWER+: CONN_01X01, MyLib:Keystone_terminal, symbol CONN_01X01
- CN1: Parts_Per_Reel 6600 -> (none)
- D3: Parts_Per_Reel 2500 -> (none); Reel_Part_No CLM1B-AKW-CUAVB253TR-ND -> (none)
- FAN: renamed from FAN1; Parts_Per_Reel -NA- -> (none); Reel_Part_No -NA- -> (none)
- JP1: Parts_Per_Reel None -> (none); Reel_Part_No None -> (none)
- POWER-: renamed from POWER-1; footprint MyLib:Keystone_4966 -> MyLib:Keystone_terminal; Parts_Per_Reel NA -> (none); Reel_Part_No NA -> (none); Supplyer_Link http://www.digikey.com/product-detail/en/keystone-electroni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 -> http://www.digikey.com/products/en?keywords=36-8197-ND; Supplyer_Part_No 36-4966-ND -> 36-8197-ND; mfr_num 4966 -> 8197
- Q1: footprint TO_SOT_Packages_SMD:TO-263-3Lead -> MyLib:TO-263-2Lead_(Small_Heat_Sink); Supplyer_Link http://www.digikey.com/product-detail/en/infineon-technolog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 -> https://www.digikey.com/product-detail/en/infineon-technolo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
- R1: Cost .1 -> (none); Parts_Per_Reel 5000 -> (none); Reel_Part_No 311-1.00KFRTR-ND -> (none)
- R2: Cost .1 -> (none); Parts_Per_Reel 5000 -> (none); Reel_Part_No 311-1.80FRTR-ND -> (none)
- R3: Cost .1 -> (none); Parts_Per_Reel 5000 -> (none); Reel_Part_No 311-300ERTR-ND -> (none)
- R4: Cost .1 -> (none); Parts_Per_Reel 5000 -> (none); Reel_Part_No 311-1.69KFRTR-ND -> (none)
- R5: Parts_Per_Reel 5000 -> (none); Reel_Part_No 311-3.60FRTR-ND -> (none)
- U1: footprint MyLib:SOP-4 -> MyLib:OP_Hybrid; symbol LTV-356T -> TLP182; Parts_Per_Reel 3500 -> (none); Reel_Part_No PS2801C-1-F3-ATR-ND -> (none)
Connections:
- wire segments 27 -> 28
Other:
- moved on the sheet: D3
